File: AC-DC Converter/AC-DC Converter.kicad_sch (KiCad schematic)
At the start: 10 parts, among them J1 Screw_Terminal_01x02, J2 Screw_Terminal_01x02

Commit message: Complete PCB routing
Parts:
- renumbered D3 to D2, D2 to D3
Other:
- note added: "12v AC to DC Converter"
Changed lines of the file:
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@@
 		(company "ZenithCore")
+	)
+	(rectangle
+		(start 52.07 44.45)
+		(end 229.87 132.08)
+		(stroke
+			(width 0)
+			(type default)
+		)
+		(fill
+			(type none)
+		)
+	)
+	(text ""
+		(exclude_from_sim no)
+		(at 80.264 58.928 0)
+		(effects
+			(font
+				(size 250 250)
+				(thickness 0.254)
+				(bold yes)
+			)
+		)
+	)
+	(text "12v AC to DC Converter"
+		(exclude_from_sim no)
+		(at 104.648 50.546 0)
+		(effects
+			(font
+				(face "Lucida Sans Typewriter")
+				(size 2.54 2.54)
+				(bold yes)
+				(italic yes)
+				(color 255 1 35 1)
+			)
+			(justify right)
+		)
 	)
 	(junction
@@
 		(dnp no)
 		(fields_autoplaced yes)
-		(property "Reference" "D3"
+		(property "Reference" "D2"
 			(at 104.14 93.98 0)
 			(show_name no)
@@
 			(project "AC-DC Converter"
 				(path "/912c8302-af48-4a23-b965-3a576f4cfed2"
-					(reference "D3")
+					(reference "D2")
 					(unit 1)
 				)
@@
 		(dnp no)
 		(fields_autoplaced yes)
-		(property "Reference" "D2"
+		(property "Reference" "D3"
 			(at 123.19 74.93 0)
 			(show_name no)
@@
 			(project "AC-DC Converter"
 				(path "/912c8302-af48-4a23-b965-3a576f4cfed2"
-					(reference "D2")
+					(reference "D3")
 					(unit 1)
 				)
