File: Transformerless Power Supply/Transformerless Power Supply.kicad_sch (KiCad schematic)
At the start: 18 parts, among them J1 Screw_Terminal_01x02, J2 Screw_Terminal_01x02, U1 LM7805_TO220

Commit message: Updated the PCB file
Parts:
- C1: footprint Package_SO:SOIC-8_3.9x4.9mm_P1.27mm -> Capacitor_THT:C_Disc_D3.4mm_W2.1mm_P2.50mm
- C2, C3: footprint (none) -> Capacitor_THT:CP_Radial_Tantal_D10.5mm_P5.00mm
- C4: footprint Package_SO:SOIC-8_3.9x4.9mm_P1.27mm -> Capacitor_THT:C_Rect_L18.0mm_W6.0mm_P15.00mm_FKS3_FKP3
- D5: footprint LED_SMD:LED_Cree-XHP50_3V_HighDensity -> LED_THT:LED_D5.0mm
- D6, D7: footprint Package_DIP:DIP-40_W15.24mm -> Diode_THT:D_A-405_P7.62mm_Horizontal
- J1, J2: footprint Package_SON:WSON-8-1EP_6x5mm_P1.27mm_EP3.4x4mm -> TerminalBlock_Wuerth:Wuerth_691311400102_P7.62mm
- R1, R2, R3, R4: footprint (none) -> Resistor_THT:R_Axial_DIN0207_L6.3mm_D2.5mm_P7.62mm_Horizontal
Connections:
- net GND: now reaches C1.2, C2.2, C3.2, D2.2 (A), D4.2 (A), D5.1 (K), J2.2 (Pin_2), R1.2, R2.2, U1.2 (GND)
- net 5v: now reaches C3.1, J2.1 (Pin_1), U1.3 (VO)
Other:
- moved on the sheet: J1, U1
